Commit message: Add moveit.launch.py to test planning with fake robot

File: stretch_moveit2/urdf/stretch_base.ros2_control.xacro (robot description, xacro)
@@ -12,4 +12,12 @@
                 <state_interface name="velocity"/>
             </joint>
+            <joint name="joint_left_wheel">
+                <state_interface name="position"/>
+                <state_interface name="velocity"/>
+            </joint>
+            <joint name="joint_right_wheel">
+                <state_interface name="position"/>
+                <state_interface name="velocity"/>
+            </joint>
         </ros2_control>
     </xacro:macro>
