Commit message: Ros World changes

File: stretch_description/urdf/stretch_aruco.xacro (robot description, xacro)
@@ -114,5 +114,5 @@
         rpy="0 0 0" />
       <mass
-        value="0" />
+        value="0.0000399141592653546" />
       <inertia
         ixx="0"
@@ -167,5 +167,5 @@
         rpy="0 0 0" />
       <mass
-        value="0" />
+        value="0.00000224999999999975" />
       <inertia
         ixx="0"
@@ -220,5 +220,5 @@
         rpy="0 0 0" />
       <mass
-        value="0" />
+        value="0.00000225" />
       <inertia
         ixx="0"

File: stretch_description/urdf/stretch_d435i.xacro (robot description, xacro)
@@ -4,9 +4,4 @@
   <xacro:arg name="add_plug" default="false"/>
   <xacro:include filename="$(find realsense2_description)/urdf/_d435i.urdf.xacro"/>
-  <!-- xyz = "
-       depth (- recessed into head / + protruding from front)
-       up and down (- down / + up)
-       sideways (- right / + left)
-       " -->
   <xacro:sensor_d435i parent="link_head_tilt" use_nominal_extrinsics="$(arg use_nominal_extrinsics)">
     <origin

File: stretch_description/urdf/stretch_description.xacro (robot description, xacro)
@@ -1,4 +1,5 @@
 <?xml version="1.0"?>
 <robot xmlns:xacro="http://www.ros.org/wiki/xacro" name="stretch_description">
+  <xacro:arg name="realsense" default="true"/>
   <xacro:include filename="stretch_gripper.xacro" />
   <!--<xacro:include filename="stretch_gripper_with_puller.xacro" />-->
@@ -6,6 +7,8 @@
   <xacro:include filename="stretch_main.xacro" />
   <xacro:include filename="stretch_aruco.xacro" />
-  <xacro:include filename="stretch_d435i.xacro" />
   <xacro:include filename="stretch_laser_range_finder.xacro" />
   <xacro:include filename="stretch_respeaker.xacro" />
+  <xacro:if value="$(arg realsense)">
+    <xacro:include filename="stretch_d435i.xacro" />
+  </xacro:if>
 </robot>

File: stretch_description/urdf/stretch_gripper.xacro (robot description, xacro)
@@ -2,4 +2,8 @@
 <robot xmlns:xacro="http://www.ros.org/wiki/xacro" name="stretch_gripper">
   <xacro:property name="scale_finger_length" value="0.9" />
+  <xacro:property name="gripper_joint_damping" value="5.75"/>
+  <xacro:property name="gripper_joint_friction" value="5.48"/>
+  <xacro:property name="gripper_joint_spring_stiffness" value="0"/>
+  <xacro:property name="gripper_joint_spring_reference" value="0"/>
   <link
     name="link_gripper">
@@ -9,5 +13,5 @@
         rpy="0 0 0" />
       <mass
-        value="0.101902711393094" />
+        value="0.000101902711393094" />
       <inertia
         ixx="0.001"
@@ -24,24 +28,17 @@
       <geometry>
         <mesh
+          filename="package://stretch_description/meshes/link_gripper.dae" />
+      </geometry>
+    </visual>
+    <collision>
+      <origin
+        xyz="0 0 0"
+        rpy="0 0 0" />
+      <geometry>
+        <mesh
           filename="package://stretch_description/meshes/link_gripper.STL" />
       </geometry>
-      <material
-        name="">
-        <color
-          rgba="0.792156862745098 0.819607843137255 0.933333333333333 1" />
-      </material>
-    </visual>
-    <collision>
-      <origin
-        xyz="0 0 0"
-        rpy="0 0 0" />
-      <geometry>
-        <mesh
-          filename="package://stretch_description/meshes/link_gripper.STL" />
-      </geometry>
-    </collision>
-  </link>
-  <!-- rpy="3.1416 0 1.5708" -->
-  <!-- rpy="0.0 0 1.5708" -->
+    </collision>
+  </link>
   <joint
     name="joint_gripper"
@@ -64,5 +61,5 @@
         rpy="0 0 0" />
       <mass
-        value="0.0476207785199474" />
+        value="0.000476207785199474" />
       <inertia
         ixx="0.001"
@@ -79,11 +76,6 @@
       <geometry>
         <mesh
-          filename="package://stretch_description/meshes/link_gripper_finger_left.STL" scale="${scale_finger_length} 1.0 1.0"/>
-      </geometry>
-      <material
-        name="">
-        <color
-          rgba="0.792156862745098 0.819607843137255 0.933333333333333 1" />
-      </material>
+          filename="package://stretch_description/meshes/link_gripper_finger_left.dae" scale="${scale_finger_length} 1.0 1.0"/>
+      </geometry>
     </visual>
     <collision>
@@ -110,6 +102,7 @@
       xyz="0 0 1" />
     <limit effort="100" lower="-0.6" upper="0.6" velocity="1.0"/>
-  </joint>
-  <link
+    <dynamics damping="${gripper_joint_damping}" friction="${gripper_joint_friction}" spring_reference="${gripper_joint_spring_reference}" spring_stiffness="{gripper_joint_spring_stiffness}"/>
+  </joint>
+  <!-- <link
     name="link_gripper_fingertip_left">
     <inertial>
@@ -118,26 +111,21 @@
         rpy="0 0 0" />
       <mass
-        value="0.00382159917455729" />
-      <inertia
-        ixx="0.001"
-        ixy="0"
-        ixz="0"
-        iyy="0.001"
-        iyz="0"
-        izz="0.001" />
-    </inertial>
-    <visual>
-      <origin
-        xyz="0 0 0"
-        rpy="0 0 0" />
-      <geometry>
-        <mesh
-          filename="package://stretch_description/meshes/link_gripper_fingertip_left.STL" />
-      </geometry>
-      <material
-        name="">
-        <color
-          rgba="0.250980392156863 0.250980392156863 0.250980392156863 1" />
-      </material>
+        value="0.000382159917455729" />
+        <inertia
+        ixx="0.001"
+        ixy="0"
+        ixz="0"
+        iyy="0.001"
+        iyz="0"
+        izz="0.001" />
+    </inertial>
+    <visual>
+      <origin
+        xyz="0 0 0"
+        rpy="0 0 0" />
+      <geometry>
+        <mesh
+          filename="package://stretch_description/meshes/link_gripper_fingertip_left.dae" />
+      </geometry>
     </visual>
     <collision>
@@ -163,5 +151,5 @@
     <axis
       xyz="0 0 0" />
-  </joint>
+  </joint> -->
   <link
     name="link_gripper_finger_right">
@@ -171,26 +159,21 @@
         rpy="0 0 0" />
       <mass
-        value="0.0476207785199481" />
-      <inertia
-        ixx="0.001"
-        ixy="0"
-        ixz="0"
-        iyy="0.001"
-        iyz="0"
-        izz="0.001" />
-    </inertial>
-    <visual>
-      <origin
-        xyz="0 0 0"
-        rpy="0 0 0" />
-      <geometry>
-        <mesh
-          filename="package://stretch_description/meshes/link_gripper_finger_right.STL" scale="${scale_finger_length} 1.0 1.0"/>
-      </geometry>
-      <material
-        name="">
-        <color
-          rgba="0.792156862745098 0.819607843137255 0.933333333333333 1" />
-      </material>
+        value="0.000476207785199481" />
+        <inertia
+        ixx="0.001"
+        ixy="0"
+        ixz="0"
+        iyy="0.001"
+        iyz="0"
+        izz="0.001" />
+    </inertial>
+    <visual>
+      <origin
+        xyz="0 0 0"
+        rpy="0 0 0" />
+      <geometry>
+        <mesh
+          filename="package://stretch_description/meshes/link_gripper_finger_right.dae" scale="${scale_finger_length} 1.0 1.0"/>
+      </geometry>
     </visual>
     <collision>
@@ -217,6 +200,7 @@
       xyz="0 0 1" />
     <limit effort="100" lower="-0.6" upper="0.6" velocity="1.0"/>
-  </joint>
-  <link
+    <dynamics damping="${gripper_joint_damping}" friction="${gripper_joint_friction}" spring_reference="${gripper_joint_spring_reference}" spring_stiffness="{gripper_joint_spring_stiffness}"/>
+  </joint>
+  <!-- <link
     name="link_gripper_fingertip_right">
     <inertial>
@@ -225,5 +209,5 @@
         rpy="0 0 0" />
       <mass
-        value="0.00382160037319545" />
+        value="0.000382160037319545" />
       <inertia
         ixx="0.001"
@@ -240,11 +224,6 @@
       <geometry>
         <mesh
-          filename="package://stretch_description/meshes/link_gripper_fingertip_right.STL" />
-      </geometry>
-      <material
-        name="">
-        <color
-          rgba="0.250980392156863 0.250980392156863 0.250980392156863 1" />
-      </material>
+          filename="package://stretch_description/meshes/link_gripper_fingertip_right.dae" />
+      </geometry>
     </visual>
     <collision>
@@ -270,5 +249,5 @@
     <axis
       xyz="0 0 0" />
-  </joint>
+  </joint> -->
   <link
       name="link_grasp_center">

File: stretch_description/urdf/stretch_laser_range_finder.xacro (robot description, xacro)
@@ -23,11 +23,6 @@
       <geometry>
         <mesh
-          filename="package://stretch_description/meshes/laser.STL" />
+          filename="package://stretch_description/meshes/laser.dae" />
       </geometry>
-      <material
-        name="">
-        <color
-          rgba="0.250980392156863 0.250980392156863 0.250980392156863 1" />
-      </material>
     </visual>
     <collision>

File: stretch_description/urdf/stretch_main.xacro (robot description, xacro)
@@ -6,4 +6,8 @@
   <xacro:property name="joint_spring_stiffness" value="0"/>
   <xacro:property name="joint_spring_reference" value="0"/>
+  <xacro:property name="caster_damping" value="0.005"/>
+  <xacro:property name="caster_friction" value="0.001"/>
+  <xacro:property name="caster_velocity_limit" value="5.0"/>
+  <xacro:property name="caster_effort_limit" value="100"/>
   <link
     name="base_link">
@@ -28,20 +32,15 @@
       <geometry>
         <mesh
+          filename="package://stretch_description/meshes/base_link.dae" />
+      </geometry>
+    </visual>
+    <collision>
+      <origin
+        xyz="0 0 0"
+        rpy="0 0 0" />
+      <geometry>
+        <mesh
           filename="package://stretch_description/meshes/base_link.STL" />
       </geometry>
-      <material
-        name="">
-        <color
-          rgba="0.792156862745098 0.819607843137255 0.933333333333333 1" />
-      </material>
-    </visual>
-    <collision>
-      <origin
-        xyz="0 0 0"
-        rpy="0 0 0" />
-      <geometry>
-        <mesh
-          filename="package://stretch_description/meshes/base_link.STL" />
-      </geometry>
     </collision>
   </link>
@@ -53,26 +52,21 @@
         rpy="0 0 0" />
       <mass
-        value="0.01" />
-      <inertia
-        ixx="0.001"
-        ixy="0"
-        ixz="0"
-        iyy="0.001"
-        iyz="0"
-        izz="0.001" />
-    </inertial>
-    <visual>
-      <origin
-        xyz="0 0 0"
-        rpy="0 0 0" />
-      <geometry>
-        <mesh
-          filename="package://stretch_description/meshes/link_right_wheel.STL" />
-      </geometry>
-      <material
-        name="">
-        <color
-          rgba="0.792156862745098 0.819607843137255 0.933333333333333 1" />
-      </material>
+        value="0.00356714564938475" />
+      <inertia
+        ixx="0.001"
+        ixy="0"
+        ixz="0"
+        iyy="0.001"
+        iyz="0"
+        izz="0.001" />
+    </inertial>
+    <visual>
+      <origin
+        xyz="0 0 0"
+        rpy="0 0 0" />
+      <geometry>
+        <mesh
+          filename="package://stretch_description/meshes/link_right_wheel.dae" />
+      </geometry>
     </visual>
     <collision>
@@ -98,5 +92,5 @@
     <axis
       xyz="0 0 1" />
-    <dynamics damping="${joint_damping}" friction="${joint_friction}" spring_reference="${joint_spring_reference}" spring_stiffness="{joint_spring_stiffness}"/>
+      <dynamics damping="${joint_damping}" friction="${joint_friction}" spring_reference="${joint_spring_reference}" spring_stiffness="{joint_spring_stiffness}"/>
   </joint>
   <link
@@ -107,26 +101,21 @@
         rpy="0 0 0" />
       <mass
-        value="0.01" />
-      <inertia
-        ixx="0.001"
-        ixy="0"
-        ixz="0"
-        iyy="0.001"
-        iyz="0"
-        izz="0.001" />
-    </inertial>
-    <visual>
-      <origin
-        xyz="0 0 0"
-        rpy="0 0 0" />
-      <geometry>
-        <mesh
-          filename="package://stretch_description/meshes/link_left_wheel.STL" />
-      </geometry>
-      <material
-        name="">
-        <color
-          rgba="0.792156862745098 0.819607843137255 0.933333333333333 1" />
-      </material>
+        value="0.00356714564938459" />
+      <inertia
+        ixx="0.001"
+        ixy="0"
+        ixz="0"
+        iyy="0.001"
+        iyz="0"
+        izz="0.001" />
+    </inertial>
+    <visual>
+      <origin
+        xyz="0 0 0"
+        rpy="0 0 0" />
+      <geometry>
+        <mesh
+          filename="package://stretch_description/meshes/link_left_wheel.dae" />
+      </geometry>
     </visual>
     <collision>
@@ -152,7 +141,48 @@
     <axis
       xyz="0 0 1" />
-    <dynamics damping="${joint_damping}" friction="${joint_friction}" spring_reference="${joint_spring_reference}" spring_stiffness="{joint_spring_stiffness}"/>
-  </joint>
-  <link name="caster_link">
+      <dynamics damping="${joint_damping}" friction="${joint_friction}" spring_reference="${joint_spring_reference}" spring_stiffness="{joint_spring_stiffness}"/>
+  </joint>
+  <!-- Representing a ball joint -->
+  <!-- <joint name="caster_joint_theta" type="continuous">
+    <origin xyz="-0.245 0.0 0.032" rpy="${-M_PI/2} 0 0"/>
+    <parent link="base_link"/>
+    <child link="caster_link_theta"/>
+    <axis xyz="0 1 0" />
+    <dynamics friction="${caster_friction}" damping="${caster_damping}" />
+    <limit lower="${-pi/2}" upper="${-pi/2}" velocity="${caster_velocity_limit}" effort="${caster_effort_limit}" />
+  </joint>
+  <link name="caster_link_theta">
+    <inertial>
+      <mass value="0.0025" />
+      <inertia ixx="5.8083e-4" ixy="0" ixz="0" iyy="3.0833e-5" iyz="0" izz="5.9083e-4" />
+    </inertial>
+  </link>
+  <joint name="caster_joint_psi" type="continuous">
+    <parent link="caster_link_theta"/>
+    <child link="caster_link_psi"/>
+    <axis xyz="0 0 1" />
+    <dynamics friction="${caster_friction}" damping="${caster_damping}" />
+    <limit lower="${-pi/2}" upper="${-pi/2}" velocity="${caster_velocity_limit}" effort="${caster_effort_limit}" />
+  </joint>
+  <link name="caster_link_psi">
+    <inertial>
+      <mass value="0.0025" />
+      <inertia ixx="5.8083e-4" ixy="0" ixz="0" iyy="3.0833e-5" iyz="0" izz="5.9083e-4" />
+    </inertial>
+  </link>
+  <joint name="caster_joint_phi" type="continuous">
+    <parent link="caster_link_theta"/>
+    <child link="caster_link_phi"/>
+    <axis xyz="1 0 0" />
+    <dynamics friction="${caster_friction}" damping="${caster_damping}" />
+  </joint>
+  <link name="caster_link_phi">
+    <inertial>
+      <mass value="0.0025" />
+      <inertia ixx="5.8083e-4" ixy="0" ixz="0" iyy="3.0833e-5" iyz="0" izz="5.9083e-4" />
+      <limit lower="${-pi/2}" upper="${-pi/2}" velocity="${caster_velocity_limit}" effort="${caster_effort_limit}" />
+    </inertial>
+  </link> -->
+  <link name="link_caster">
     <collision>
       <geometry>
@@ -169,4 +199,13 @@
           </ode>
         </friction>
+        <contact>
+          <ode>
+            <soft_cfm>0</soft_cfm>
+            <soft_erp>0.2</soft_erp>
+            <kp>1e+13</kp>
+            <kd>1</kd>
+            <min_depth>0.001</min_depth>
+          </ode>
+        </contact>
       </surface>
     </collision>
@@ -177,11 +216,6 @@
       <geometry>
         <mesh
-          filename="package://stretch_description/meshes/omni_wheel_m.STL" />
-      </geometry>
-      <material
-        name="">
-        <color
-          rgba="0.792156862745098 0.819607843137255 0.933333333333333 1" />
-      </material>
+          filename="package://stretch_description/meshes/omni_wheel_m.dae" />
+      </geometry>
     </visual>
     <inertial>
@@ -197,9 +231,9 @@
     </inertial>
   </link>
-  <joint name="caster_joint" type="fixed">
+  <joint name="joint_caster" type="fixed">
+    <!-- <parent link="caster_link_phi"/> -->
     <parent link="base_link"/>
-    <child link="caster_link"/>
+    <child link="link_caster"/>
     <origin xyz="-0.245 0.0 0.032" rpy="${-M_PI/2} 0 0"/>
-    <axis xyz="0 0 1" />
   </joint>
   <link
@@ -207,29 +241,24 @@
     <inertial>
       <origin
-        xyz="0.00755818572975822 0.773971284176834 0.00647313086620024"
-        rpy="0 0 0" />
-      <mass
-        value="0.749143203376401" />
-      <inertia
-        ixx="0.0709854511954588"
-        ixy="-0.00433428742758457"
-        ixz="-0.000186110788697573"
-        iyy="0.000437922053342648"
-        iyz="-0.00288788257713431"
-        izz="0.071104808501661" />
-    </inertial>
-    <visual>
-      <origin
-        xyz="0 0 0"
-        rpy="0 0 0" />
-      <geometry>
-        <mesh
-          filename="package://stretch_description/meshes/link_mast.STL" />
-      </geometry>
-      <material
-        name="">
-        <color
-          rgba="0.792156862745098 0.819607843137255 0.933333333333333 1" />
-      </material>
+        xyz="-0.109461304328163 -0.000741018909047708 0.0914915269429946"
+        rpy="0 0 0" />
+      <mass
+        value="0.05" />
+      <inertia
+        ixx="0.001"
+        ixy="0.0"
+        ixz="0.0"
+        iyy="0.001"
+        iyz="0.0"
+        izz="0.001" />
+    </inertial>
+    <visual>
+      <origin
+        xyz="0 0 0"
+        rpy="0 0 0" />
+      <geometry>
+        <mesh
+          filename="package://stretch_description/meshes/link_mast.dae" />
+      </geometry>
     </visual>
     <collision>
@@ -263,26 +292,21 @@
         rpy="0 0 0" />
       <mass
-        value="0.444820831236007" />
-      <inertia
-        ixx="0.000567192946271367"
-        ixy="-0.00024607534789508"
-        ixz="-0.000128108442260574"
-        iyy="0.00127108364478659"
-        iyz="7.61916855070339E-06"
-        izz="0.00137296635099006" />
-    </inertial>
-    <visual>
-      <origin
-        xyz="0 0 0"
-        rpy="0 0 0" />
-      <geometry>
-        <mesh
-          filename="package://stretch_description/meshes/link_lift.STL" />
-      </geometry>
-      <material
-        name="">
-        <color
-          rgba="0.792156862745098 0.819607843137255 0.933333333333333 1" />
-      </material>
+        value="0.044820831236007" />
+      <inertia
+        ixx="0.001"
+        ixy="0.0"
+        ixz="0.0"
+        iyy="0.001"
+        iyz="0.0"
+        izz="0.001" />
+    </inertial>
+    <visual>
+      <origin
+        xyz="0 0 0"
+        rpy="0 0 0" />
+      <geometry>
+        <mesh
+          filename="package://stretch_description/meshes/link_lift.dae" />
+      </geometry>
     </visual>
     <collision>
@@ -300,5 +324,5 @@
     type="prismatic">
     <origin
-      xyz="-0.0369217062323472 0.165471199999996 -0.000341653286793524"
+      xyz="-0.0369217062323472 0.266771199999996 -0.000341653286793524"
       rpy="-1.57079632679552 1.5615431375292 -6.2942004366467E-13" />
     <parent
@@ -307,9 +331,8 @@
       link="link_lift" />
     <axis
-	xyz="0 0 1" />
-  <!-- for now, hand copied range_m from lift (from ~/repos/stretch_fleet/stretch-re1-1001/stretch_re1_factory_params.yaml) -->
-  <!--<limit effort="100" lower="0.0" upper="1.095" velocity="1.0"/>-->
-  <!-- copied value did not reach the top of mesh model with GUI sliders and RViz -->
-  <limit effort="100" lower="0.0" upper="1.1" velocity="1.0"/>
+  xyz="0 0 1" />
+    <limit effort="100" lower="-0.1033" upper="0.9967" velocity="1.0"/>
+    <!-- Make this high friction so gripper does not fall -->
+    <dynamics damping="10" friction="10.48" spring_reference="${joint_spring_reference}" spring_stiffness="{joint_spring_stiffness}"/>
   </joint>
   <link
@@ -320,26 +343,21 @@
         rpy="0 0 0" />
       <mass
-        value="0.0676525455789735" />
-      <inertia
-        ixx="0.000122002023066796"
-        ixy="7.29593356230121E-13"
-        ixz="9.63170353371061E-09"
-        iyy="0.000122002023127152"
-        iyz="-9.24154949889042E-09"
-        izz="1.46043439809638E-12" />
-    </inertial>
-    <visual>
-      <origin
-        xyz="0 0 0"
-        rpy="0 0 0" />
-      <geometry>
-        <mesh
-          filename="package://stretch_description/meshes/link_arm_l4.STL" />
-      </geometry>
-      <material
-        name="">
-        <color
-          rgba="0.792156862745098 0.819607843137255 0.933333333333333 1" />
-      </material>
+        value="0.00676525455789735" />
+      <inertia
+        ixx="0.001"
+        ixy="0"
+        ixz="0"
+        iyy="0.001"
+        iyz="0"
+        izz="0.001" />
+    </inertial>
+    <visual>
+      <origin
+        xyz="0 0 0"
+        rpy="0 0 0" />
+      <geometry>
+        <mesh
+          filename="package://stretch_description/meshes/link_arm_l4.dae" />
+      </geometry>
     </visual>
     <collision>
@@ -373,26 +391,21 @@
         rpy="0 0 0" />
       <mass
-        value="0.0626921047058405" />
-      <inertia
-        ixx="0.001"
-        ixy="0"
-        ixz="0"
-        iyy="0.001"
-        iyz="0"
-        izz="0.001" />
-    </inertial>
-    <visual>
-      <origin
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