Commit message: revert URDF changes

File: stretch_description/urdf/stretch_aruco.xacro (robot description, xacro)
@@ -5,5 +5,5 @@
     <inertial>
       <origin
-        xyz="1.3878E-17 0 -0.000125"
+        xyz="0 0 -5.00000000014378E-07"
         rpy="0 0 0" />
       <mass
@@ -45,5 +45,5 @@
     type="fixed">
     <origin
-      xyz="-0.0015028 -0.1304972 0.1597482"
+      xyz="-0.00500000000000014 -0.1304972 0.1597482"
       rpy="0 0 -1.5707963267949" />
     <parent
@@ -58,5 +58,5 @@
     <inertial>
       <origin
-        xyz="2.7756E-17 0 -0.000125"
+        xyz="0 0 -5.00000000014378E-07"
         rpy="0 0 0" />
       <mass
@@ -164,5 +164,5 @@
     <inertial>
       <origin
-        xyz="-1.3531E-15 -3.4972E-15 -0.000125"
+        xyz="1.11022302462516E-16 3.05311331771918E-16 -0.00012499999999821"
         rpy="0 0 0" />
       <mass

File: stretch_description/urdf/stretch_laser_range_finder.xacro (robot description, xacro)
@@ -45,6 +45,6 @@
     type="fixed">
     <origin
-      xyz="0.004 0 0.1664"
-      rpy="0 0 3.1416" />
+      xyz="0.000502800000000914 0 0.1664"
+      rpy="0 0 -3.14159265358979" />
     <parent
       link="base_link" />

File: stretch_description/urdf/stretch_main.xacro (robot description, xacro)
@@ -10,15 +10,15 @@
     <inertial>
       <origin
-        xyz="-0.11587 0.0019426 0.093621"
-        rpy="0 0 0" />
-      <mass
-        value="1.1912" />
-      <inertia
-        ixx="0.0034667"
-        ixy="-5.0568E-06"
-        ixz="0.00042861"
-        iyy="0.0052744"
-        iyz="-5.766E-05"
-        izz="0.0047945" />
+        xyz="-0.109461304328163 -0.000741018909047708 0.0914915269429946"
+        rpy="0 0 0" />
+      <mass
+        value="1.0723782659782" />
+      <inertia
+        ixx="0.00310580907710135"
+        ixy="1.5182848191076E-06"
+        ixz="0.00041690466732394"
+        iyy="0.00433798719991832"
+        iyz="1.33487716258445E-05"
+        izz="0.0037204727467362" />
     </inertial>
     <visual>
@@ -33,5 +33,5 @@
         name="">
         <color
-          rgba="0.79216 0.81961 0.93333 1" />
+          rgba="0.792156862745098 0.819607843137255 0.933333333333333 1" />
       </material>
     </visual>
@@ -50,8 +50,8 @@
     <inertial>
       <origin
-        xyz="1.1719E-11 2.0783E-11 0.037544"
-        rpy="0 0 0" />
-      <mass
-        value="0.0042721" />
+        xyz="1.25554620866719E-07 3.54748938447003E-07 0.0239581106165018"
+        rpy="0 0 0" />
+      <mass
+        value="0.01" />
       <inertia
         ixx="0.001"
@@ -73,5 +73,5 @@
         name="">
         <color
-          rgba="0.79216 0.81961 0.93333 1" />
+          rgba="0.792156862745098 0.819607843137255 0.933333333333333 1" />
       </material>
     </visual>
@@ -90,6 +90,6 @@
     type="continuous">
     <origin
-      xyz="0 -0.17035 0.0508"
-      rpy="-1.5708 1.2717E-16 4.8006E-17" />
+      xyz="-0.00300000000000034 -0.15765 0.0508000000000004"
+      rpy="-1.57079632679489 -1.11022302462516E-16 7.28583859910277E-17" />
     <parent
       link="base_link" />
@@ -98,5 +98,5 @@
     <axis
       xyz="0 0 1" />
-    <dynamics damping="${joint_damping}" friction="${joint_friction}" spring_reference="${joint_spring_reference}" spring_stiffness="${joint_spring_stiffness}"/>
+    <dynamics damping="${joint_damping}" friction="${joint_friction}" spring_reference="${joint_spring_reference}" spring_stiffness="{joint_spring_stiffness}"/>
   </joint>
   <link
@@ -104,8 +104,8 @@
     <inertial>
       <origin
-        xyz="-2.0783E-11 -1.1719E-11 -0.037544"
-        rpy="0 0 0" />
-      <mass
-        value="0.0042721" />
+        xyz="1.2555462092223E-07 -3.54748938502514E-07 -0.0239581106165035"
+        rpy="0 0 0" />
+      <mass
+        value="0.01" />
       <inertia
         ixx="0.001"
@@ -127,5 +127,5 @@
         name="">
         <color
-          rgba="0.79216 0.81961 0.93333 1" />
+          rgba="0.792156862745098 0.819607843137255 0.933333333333333 1" />
       </material>
     </visual>
@@ -144,6 +144,6 @@
     type="continuous">
     <origin
-      xyz="0 0.17035 0.0508"
-      rpy="-1.5708 2.6317E-16 -8.2057E-19" />
+      xyz="-0.00300000000001899 0.15765 0.0507999999999994"
+      rpy="-1.5707963267949 3.16227047920818E-31 7.88745438253713E-16" />
     <parent
       link="base_link" />
@@ -152,5 +152,5 @@
     <axis
       xyz="0 0 1" />
-    <dynamics damping="${joint_damping}" friction="${joint_friction}" spring_reference="${joint_spring_reference}" spring_stiffness="${joint_spring_stiffness}"/>
+    <dynamics damping="${joint_damping}" friction="${joint_friction}" spring_reference="${joint_spring_reference}" spring_stiffness="{joint_spring_stiffness}"/>
   </joint>
   <link name="caster_link">
@@ -207,8 +207,8 @@
     <inertial>
       <origin
-        xyz="2.0817E-17 0.7075 -2.7756E-17"
-        rpy="0 0 0" />
-      <mass
-        value="1.8285" />
+        xyz="0.00755818572975822 0.773971284176834 0.00647313086620024"
+        rpy="0 0 0" />
+      <mass
+        value="0.749143203376401" />
       <inertia
         ixx="0.0709854511954588"
@@ -230,5 +230,5 @@
         name="">
         <color
-          rgba="0.79216 0.81961 0.93333 1" />
+          rgba="0.792156862745098 0.819607843137255 0.933333333333333 1" />
       </material>
     </visual>
@@ -247,6 +247,6 @@
     type="fixed">
     <origin
-      xyz="-0.067 0.135 0.0284"
-      rpy="1.5708 0 4.8006E-17" />
+      xyz="-0.07 0.134999999999998 0.0284000000000001"
+      rpy="1.5707963267949 0 0.00925318926571245" />
     <parent
       link="base_link" />
@@ -260,15 +260,15 @@
     <inertial>
       <origin
-        xyz="-0.031727 0.038403 0.013361"
-        rpy="0 0 0" />
-      <mass
-        value="0.27218" />
-      <inertia
-        ixx="0.00052571"
-        ixy="0.00014899"
-        ixz="-1.9258E-05"
-        iyy="0.00030679"
-        iyz="-6.2451E-06"
-        izz="0.00037324" />
+        xyz="-0.0547636346252869 0.0380939689802074 0.00933159404448308"
+        rpy="0 0 0" />
+      <mass
+        value="0.444820831236007" />
+      <inertia
+        ixx="0.000567192946271367"
+        ixy="-0.00024607534789508"
+        ixz="-0.000128108442260574"
+        iyy="0.00127108364478659"
+        iyz="7.61916855070339E-06"
+        izz="0.00137296635099006" />
     </inertial>
     <visual>
@@ -283,5 +283,5 @@
         name="">
         <color
-          rgba="0.79216 0.81961 0.93333 1" />
+          rgba="0.792156862745098 0.819607843137255 0.933333333333333 1" />
       </material>
     </visual>
@@ -300,6 +300,6 @@
     type="prismatic">
     <origin
-      xyz="-0.037385 0.1666 0"
-      rpy="-1.5708 1.5708 0" />
+      xyz="-0.0369217062323472 0.165471199999996 -0.000341653286793524"
+      rpy="-1.57079632679552 1.5615431375292 -6.2942004366467E-13" />
     <parent
       link="link_mast" />
@@ -307,6 +307,6 @@
       link="link_lift" />
     <axis
-      xyz="0 0 1" />
-  <!-- for now hand copied range_m from lift from ~/repos/stretch_fleet/stretch-re1-1001/stretch_re1_factory_params.yaml -->
+	xyz="0 0 1" />
+  <!-- for now, hand copied range_m from lift (from ~/repos/stretch_fleet/stretch-re1-1001/stretch_re1_factory_params.yaml) -->
   <!--<limit effort="100" lower="0.0" upper="1.095" velocity="1.0"/>-->
   <!-- copied value did not reach the top of mesh model with GUI sliders and RViz -->
@@ -317,15 +317,15 @@
     <inertial>
       <origin
-        xyz="-1.0146E-06 -1.9719E-05 -0.094738"
-        rpy="0 0 0" />
-      <mass
-        value="0.068095" />
-      <inertia
-        ixx="0.0001256"
-        ixy="-5.6914E-12"
-        ixz="6.0647E-09"
-        iyy="0.0001256"
-        iyz="1.1787E-07"
-        izz="1.1091E-10" />
+        xyz="-1.61247276464493E-06 1.54715589201215E-06 -0.0953252706040035"
+        rpy="0 0 0" />
+      <mass
+        value="0.0676525455789735" />
+      <inertia
+        ixx="0.000122002023066796"
+        ixy="7.29593356230121E-13"
+        ixz="9.63170353371061E-09"
+        iyy="0.000122002023127152"
+        iyz="-9.24154949889042E-09"
+        izz="1.46043439809638E-12" />
     </inertial>
     <visual>
@@ -340,5 +340,5 @@
         name="">
         <color
-          rgba="0.79216 0.81961 0.93333 1" />
+          rgba="0.792156862745098 0.819607843137255 0.933333333333333 1" />
       </material>
     </visual>
@@ -357,6 +357,6 @@
     type="fixed">
     <origin
-      xyz="-0.2547 0 0"
-      rpy="1.5708 2.4721E-15 -1.5708" />
+      xyz="-0.25471 0 0"
+      rpy="1.5708 -3.1019E-16 -1.5708" />
     <parent
       link="link_lift" />
@@ -370,8 +370,8 @@
     <inertial>
       <origin
-        xyz="-5.13853606326845E-07 -1.99844969271112E-05 -0.0971104963726614"
-        rpy="0 0 0" />
-      <mass
-        value="0.0628927381893134" />
+        xyz="-3.34873468621488E-07 4.7411336306924E-07 -0.0974069598289041"
+        rpy="0 0 0" />
+      <mass
+        value="0.0626921047058405" />
       <inertia
         ixx="0.001"
@@ -411,5 +411,5 @@
     <origin
       xyz="0 0 0.013"
-      rpy="7.68831233799385E-30 2.36716479416092E-30 2.29652732251143E-17" />
+      rpy="3.5742E-16 3.2123E-16 -2.4565E-16" />
     <parent
       link="link_arm_l4" />
@@ -417,5 +417,5 @@
       link="link_arm_l3" />
     <axis
-      xyz="0 0 1" />
+	xyz="0 0 1" />
     <!-- 0.13 = 0.52/4-->
     <limit effort="100" lower="0.0" upper="0.13" velocity="1.0"/>
@@ -425,8 +425,8 @@
     <inertial>
       <origin
-        xyz="-5.17421949435687E-07 -2.02045301450349E-05 -0.0968815475684904"
-        rpy="0 0 0" />
-      <mass
-        value="0.0571386353275368" />
+        xyz="-3.31043560508615E-07 3.13422303999111E-07 -0.097255883541891"
+        rpy="0 0 0" />
+      <mass
+        value="0.0569074368576238" />
       <inertia
         ixx="0.001"
@@ -466,5 +466,5 @@
     <origin
       xyz="0 0 0.013"
-      rpy="0 1.57655765344625E-30 -1.66533453693773E-16" />
+      rpy="2.91385731014123E-16 4.44300759504684E-17 3.25691080516352E-16" />
     <parent
       link="link_arm_l3" />
@@ -472,5 +472,5 @@
       link="link_arm_l2" />
     <axis
-      xyz="0 0 1" />
+	xyz="0 0 1" />
     <!-- 0.13 = 0.52/4-->
     <limit effort="100" lower="0.0" upper="0.13" velocity="1.0"/>
@@ -480,8 +480,8 @@
     <inertial>
       <origin
-        xyz="-5.257E-07 -2.0482E-05 -0.096543"
-        rpy="0 0 0" />
-      <mass
-        value="0.051382" />
+        xyz="-3.36876635420591E-07 3.05876091066803E-07 -0.0969117032232756"
+        rpy="0 0 0" />
+      <mass
+        value="0.0511763619538321" />
       <inertia
         ixx="0.001"
@@ -503,5 +503,5 @@
         name="">
         <color
-          rgba="0.79216 0.81961 0.93333 1" />
+          rgba="0.792156862745098 0.819607843137255 0.933333333333333 1" />
       </material>
     </visual>
@@ -520,6 +520,6 @@
     type="prismatic">
     <origin
-      xyz="0 0 0.0129999999999981"
-      rpy="-7.63746778746202E-30 -7.88860905221012E-31 1.11022302462516E-16" />
+      xyz="0 0 0.013"
+      rpy="7.41596560408007E-17 1.33876788296791E-16 -2.44545873596083E-16" />
     <parent
       link="link_arm_l2" />
@@ -527,5 +527,5 @@
       link="link_arm_l1" />
     <axis
-      xyz="0 0 1" />
+	xyz="0 0 1" />
     <!-- 0.13 = 0.52/4-->
     <limit effort="100" lower="0.0" upper="0.13" velocity="1.0"/>
@@ -535,8 +535,8 @@
     <inertial>
       <origin
-        xyz="0.0270582141286185 -0.00189876414654466 -0.0377809018481181"
-        rpy="0 0 0" />
-      <mass
-        value="0.085003260946398" />
+        xyz="0.0230715049668191 -0.00195115833662818 -0.0360646347160285"
+        rpy="0 0 0" />
+      <mass
+        value="0.101241250325294" />
       <inertia
         ixx="0.001"
@@ -575,6 +575,6 @@
     type="prismatic">
     <origin
-      xyz="0 0 -0.0137499999991968"
-      rpy="7.63746778746202E-30 -3.80121128864402E-15 2.62707547767438E-15" />
+      xyz="0 0 -0.0137499999999938"
+      rpy="-3.05317390622457E-16 -4.23236224076729E-16 -2.68425135229209E-17" />
     <parent
       link="link_arm_l1" />
@@ -582,5 +582,5 @@
       link="link_arm_l0" />
     <axis
-      xyz="0 0 1" />
+	xyz="0 0 1" />
     <!-- 0.13 = 0.52/4-->
     <limit effort="100" lower="0.0" upper="0.13" velocity="1.0"/>
@@ -590,8 +590,8 @@
     <inertial>
       <origin
-        xyz="2.20122392535771E-11 2.9317167880849E-05 -0.018966592644729"
-        rpy="0 0 0" />
-      <mass
-        value="0.0404746907425003" />
+        xyz="-8.02795716750571E-06 1.93811447768422E-05 0.018946700595851"
+        rpy="0 0 0" />
+      <mass
+        value="0.0405398981326229" />
       <inertia
         ixx="0.001"
@@ -613,5 +613,5 @@
         name="">
         <color
-          rgba="0.898039215686275 0.917647058823529 0.929411764705882 1" />
+	        rgba="0.792156862745098 0.819607843137255 0.933333333333333 1" />
       </material>
     </visual>
@@ -630,6 +630,6 @@
     type="revolute">
     <origin
-      xyz="0.0830000000000654 -0.0307500000000129 0"
-      rpy="1.5708 4.2595E-14 2.6415E-15"/>
+      xyz="0.083 -0.03075 0"
+      rpy="1.5708 4.2595E-14 2.6415E-15" />
     <parent
       link="link_arm_l0" />
@@ -639,7 +639,7 @@
       xyz="0 0 -1" />
     <!--
-      stowed to front ~225 deg, 3.15159 x 1.25 = 3.9395
+      stowed to front ~225 deg (3.9395 radians)
       using 4.0
-      stowed to back ~100 deg, 100 / 180 x 3.14159 = 1.7453
+      stowed to back ~100 deg (1.7453 radians)
       using -1.75
     -->
@@ -650,8 +650,8 @@
     <inertial>
       <origin
-        xyz="0.0406850995527703 0.0396956343318414 0.0226500246461012"
-        rpy="0 0 0" />
-      <mass
-        value="0.133027236718691" />
+        xyz="0.0372933550588956 0.045509432985552 0.0281136801213409"
+        rpy="0 0 0" />
+      <mass
+        value="0.129454717596498" />
       <inertia
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
File: stretch_description/urdf/stretch_respeaker.xacro (robot description, xacro)
@@ -1,19 +1,18 @@
 <?xml version="1.0"?>
 <robot xmlns:xacro="http://www.ros.org/wiki/xacro" name="stretch_respeaker">
-  <link
-    name="respeaker_base">
+  <link name="respeaker_base">
     <inertial>
       <origin
-        xyz="-0.003809 -0.0023075 -0.012854"
+        xyz="-0.00078082896792734 0.00765742173486017 -0.0042488298301937"
         rpy="0 0 0" />
       <mass
-        value="0.015643" />
+        value="0.00969129410417277" />
       <inertia
-        ixx="1.0075E-06"
-        ixy="-5.4396E-08"
-        ixz="-2.8652E-07"
-        iyy="1.0569E-06"
-        iyz="-1.8463E-07"
-        izz="1.1947E-07" />
+        ixx="8.95656300428405E-07"
+        ixy="2.67330745809535E-08"
+        ixz="-3.84519793580934E-08"
+        iyy="4.0421099617056E-07"
+        iyz="3.15533542838673E-07"
+        izz="7.08282597118018E-07" />
     </inertial>
     <visual>
@@ -23,10 +22,10 @@
       <geometry>
         <mesh
-          filename="package://stretch_description/meshes/respeaker_base.STL" />
+          filename="package://stretch_description/meshes/link_respeaker.STL" />
       </geometry>
       <material
         name="">
         <color
-          rgba="0.79216 0.81961 0.93333 1" />
+          rgba="0.792156862745098 0.819607843137255 0.933333333333333 1" />
       </material>
     </visual>
@@ -37,5 +36,5 @@
       <geometry>
         <mesh
-          filename="package://stretch_description/meshes/respeaker_base.STL" />
+          filename="package://stretch_description/meshes/link_respeaker.STL" />
       </geometry>
     </collision>
@@ -44,7 +43,8 @@
     name="joint_respeaker"
     type="fixed">
+    <!-- rpy="   ?   rotate_sound_source_direction    ?   " -->
     <origin
-      xyz="0 1.37236408874452 0.00303065898329655"
-      rpy="-1.5707963267949 -0.698131700797725 4.93295812652799E-16" />
+      xyz="1.09074743137871E-05 1.36992 0.00303572796911382"
+      rpy="1.57079632679553 0.0 3.14159265358916" />
     <parent
       link="link_mast" />
